Commit message: Added mesh file for intel realsense D415

File: jetsoncar_ws/src/realsense2_camera/urdf/_d435.urdf.xacro (robot description, xacro)
@@ -40,6 +40,5 @@
         <geometry>
           <!-- <box size="${d435_cam_width} ${d435_cam_height} ${d435_cam_depth}"/> -->
-	  <mesh filename="package://realsense2_camera/meshes/d435.dae" />
-          <!--<mesh filename="package://realsense2_camera/meshes/d435/d435.dae" />-->
+	         <mesh filename="package://realsense2_camera/meshes/d435.dae" />
         </geometry>
         <material name="aluminum"/>
