Commit message: Working simulation with new realsense2_description package

File: jetsoncar_ws/src/realsense2_description/urdf/_d415.urdf.xacro (robot description, xacro)
@@ -40,5 +40,5 @@
         <geometry>
           <!--<box size="${d415_cam_width} ${d415_cam_height} ${d415_cam_depth}"/>-->
-          <mesh filename="package://realsense2_camera/meshes/d415.dae" />
+          <mesh filename="package://realsense2_description/meshes/d415.dae" />
         </geometry>
         <material name="aluminum"/>

File: jetsoncar_ws/src/realsense2_description/urdf/_d435.urdf.xacro (robot description, xacro)
@@ -40,5 +40,5 @@
         <geometry>
           <!-- <box size="${d435_cam_width} ${d435_cam_height} ${d435_cam_depth}"/> -->
-	         <mesh filename="package://realsense2_camera/meshes/d435.dae" />
+	         <mesh filename="package://realsense2_description/meshes/d435.dae" />
         </geometry>
         <material name="aluminum"/>
