Commit message: put intel realsense camera on the car

File: jetsoncar_ws/src/racecar_description/urdf/racecar.xacro (robot description, xacro)
@@ -149,9 +149,9 @@
   </joint>
   <xacro:wheel_transmission name="right_front_wheel" />
-  <!-- RealSense D415 Camera -->
-  <xacro:include filename="$(find realsense2_description)/urdf/_d415.urdf.xacro"/>
-  <sensor_d415 parent="chassis" camera_name="front_cam">
+  <!-- RealSense D435 Camera -->
+  <xacro:include filename="$(find realsense2_description)/urdf/_d435.urdf.xacro"/>
+  <sensor_d435 parent="chassis" camera_name="front_cam">
     <origin xyz="0.350 0 0.04" rpy="0 0 0"/>
-  </sensor_d415>
+  </sensor_d435>
   <!-- IMU -->
   <link name="imu_link">

File: jetsoncar_ws/src/realsense2_description/urdf/_d415.urdf.xacro (robot description, xacro)
@@ -52,5 +52,5 @@
       <inertial>
         <!-- The following are not reliable values, and should not be used for modeling -->
-        <mass value="0.564" />
+        <mass value="0.072" />
         <origin xyz="0 0 0" />
         <inertia ixx="0.003881243" ixy="0.0" ixz="0.0" iyy="0.000498940" iyz="0.0" izz="0.003879257" />

File: jetsoncar_ws/src/realsense2_description/urdf/_d435.urdf.xacro (robot description, xacro)
@@ -52,5 +52,5 @@
       <inertial>
         <!-- The following are not reliable values, and should not be used for modeling -->
-        <mass value="0.564" />
+        <mass value="0.072" />
         <origin xyz="0 0 0" />
         <inertia ixx="0.003881243" ixy="0.0" ixz="0.0" iyy="0.000498940" iyz="0.0" izz="0.003879257" />
